File: kicad/COM.sch (KiCad schematic (older format))
At the start: 1 part, among them J5 COM

Commit message: 部品を配置 kicad5
Parts:
- removed J5: COM, mouse:JST_SH_BM03B-SRSS-TB_03x1.00mm_Straight, symbol CONN_01X03
- added J7: COM, mouse:JST_SH_BM03B-SRSS-TB_03x1.00mm_Straight, symbol Connector:Conn_01x03_Male
Connections:
- net GND: now also J7.1 (Pin_1)
- net UART_RX: now also J7.2 (Pin_2)
- net UART_TX: now also J7.3 (Pin_3)
Changed lines of the file:
@@
-EESchema Schematic File Version 2
-LIBS:power
-LIBS:device
-LIBS:transistors
-LIBS:conn
-LIBS:linear
-LIBS:regul
-LIBS:74xx
-LIBS:cmos4000
-LIBS:adc-dac
-LIBS:memory
-LIBS:xilinx
-LIBS:microcontrollers
-LIBS:dsp
-LIBS:microchip
-LIBS:analog_switches
-LIBS:motorola
-LIBS:texas
-LIBS:intel
-LIBS:audio
-LIBS:interface
-LIBS:digital-audio
-LIBS:philips
-LIBS:display
-LIBS:cypress
-LIBS:siliconi
-LIBS:opto
-LIBS:atmel
-LIBS:contrib
-LIBS:valves
-LIBS:KERISE
-LIBS:74xgxx
-LIBS:ac-dc
-LIBS:actel
-LIBS:allegro
-LIBS:Altera
-LIBS:analog_devices
-LIBS:battery_management
-LIBS:bbd
-LIBS:bosch
-LIBS:brooktre
-LIBS:cmos_ieee
-LIBS:dc-dc
-LIBS:diode
-LIBS:elec-unifil
-LIBS:ESD_Protection
-LIBS:ftdi
-LIBS:gennum
-LIBS:hc11
-LIBS:ir
-LIBS:Lattice
-LIBS:leds
-LIBS:maxim
-LIBS:mechanical
-LIBS:microchip_dspic33dsc
-LIBS:microchip_pic10mcu
-LIBS:microchip_pic12mcu
-LIBS:microchip_pic16mcu
-LIBS:microchip_pic18mcu
-LIBS:microchip_pic24mcu
-LIBS:microchip_pic32mcu
-LIBS:modules
-LIBS:motor_drivers
-LIBS:motors
-LIBS:msp430
-LIBS:nordicsemi
-LIBS:nxp
-LIBS:nxp_armmcu
-LIBS:onsemi
-LIBS:Oscillators
-LIBS:Power_Management
-LIBS:powerint
-LIBS:pspice
-LIBS:references
-LIBS:relays
-LIBS:rfcom
-LIBS:sensors
-LIBS:silabs
-LIBS:stm8
-LIBS:stm32
-LIBS:supertex
-LIBS:switches
-LIBS:transf
-LIBS:triac_thyristor
-LIBS:ttl_ieee
-LIBS:video
-LIBS:wiznet
-LIBS:Worldsemi
-LIBS:Xicor
-LIBS:zetex
-LIBS:Zilog
-LIBS:graphic_symbols
-LIBS:infineon
-LIBS:intersil
-LIBS:LEM
-LIBS:logic_programmable
-LIBS:RFSolutions
+EESchema Schematic File Version 4
 LIBS:KERISE-cache
-EELAYER 25 0
+EELAYER 26 0
 EELAYER END
 $Descr A4 11693 8268
 encoding utf-8
-Sheet 6 15
+Sheet 6 14
 Title ""
 Date ""
@@
 $EndDescr
 $Comp
-L GND #PWR042
+L power:GND #PWR039
 U 1 1 57CDAC76
 P 4800 4200
-F 0 "#PWR042" H 4800 3950 50  0001 C CNN
+F 0 "#PWR039" H 4800 3950 50  0001 C CNN
 F 1 "GND" H 4800 4050 50  0000 C CNN
 F 2 "" H 4800 4200 50  0000 C CNN
@@
 COM Port
 $Comp
-L CONN_01X03 J5
-U 1 1 59807C31
+L Connector:Conn_01x03_Male J7
+U 1 1 5B6F3423
 P 4500 4000
-F 0 "J5" H 4500 4200 50  0000 C CNN
-F 1 "COM" V 4600 4000 50  0000 C CNN
+F 0 "J7" H 4606 4278 50  0000 C CNN
+F 1 "COM" H 4606 4187 50  0000 C CNN
 F 2 "mouse:JST_SH_BM03B-SRSS-TB_03x1.00mm_Straight" H 4500 4000 50  0001 C CNN
-F 3 "" H 4500 4000 50  0001 C CNN
+F 3 "~" H 4500 4000 50  0001 C CNN
 	1    4500 4000
-	-1   0    0    -1
+	1    0    0    -1
 $EndComp
 $EndSCHEMATC
