File: kicad/Encoder.sch (KiCad schematic (older format))
At the start: 4 parts, among them P5 ENC_Host, P6 ENC_Slave, U6 AS5048A

Commit message: 回路を改良
受光部をフォトトランジスタに変更
測距センサをVL6180Xに変更
動作電圧を3Vに変更
Parts:
- P5: footprint mouse:STAND_AS_HOST -> mouse:STAND_HOST_06
- P6: footprint mouse:STAND_AS_SLAVE -> mouse:STAND_SLAVE_06
- renumbered C16 to C10, U6 to U4
Changed lines of the file:
@@
 LIBS:ftdi
 LIBS:gennum
-LIBS:graphic
 LIBS:hc11
 LIBS:ir
 LIBS:Lattice
 LIBS:leds
-LIBS:logo
 LIBS:maxim
 LIBS:mechanical
@@
 LIBS:zetex
 LIBS:Zilog
+LIBS:graphic_symbols
+LIBS:infineon
+LIBS:intersil
+LIBS:LEM
+LIBS:logic_programmable
+LIBS:RFSolutions
 LIBS:KERISE-cache
 EELAYER 25 0
@@
 $EndDescr
 $Comp
-L GND #PWR050
+L GND #PWR048
 U 1 1 589E94E9
 P 4100 3600
-AR Path="/592ADBF2/589E94E9" Ref="#PWR050"  Part="1"
-AR Path="/59347BCD/589E94E9" Ref="#PWR058"  Part="1"
-F 0 "#PWR058" H 4100 3350 50  0001 C CNN
+AR Path="/592ADBF2/589E94E9" Ref="#PWR048"  Part="1"
+AR Path="/59347BCD/589E94E9" Ref="#PWR056"  Part="1"
+F 0 "#PWR056" H 4100 3350 50  0001 C CNN
 F 1 "GND" H 4100 3450 50  0000 C CNN
 F 2 "" H 4100 3600 50  0000 C CNN
@@
 CS
 $Comp
-L PWR_FLAG #FLG051
+L PWR_FLAG #FLG049
 U 1 1 58CB39A3
 P 5100 2900
-AR Path="/592ADBF2/58CB39A3" Ref="#FLG051"  Part="1"
-AR Path="/59347BCD/58CB39A3" Ref="#FLG059"  Part="1"
-F 0 "#FLG059" H 5100 2995 50  0001 C CNN
+AR Path="/592ADBF2/58CB39A3" Ref="#FLG049"  Part="1"
+AR Path="/59347BCD/58CB39A3" Ref="#FLG057"  Part="1"
+F 0 "#FLG057" H 5100 2995 50  0001 C CNN
 F 1 "PWR_FLAG" H 5100 3080 50  0000 C CNN
 F 2 "" H 5100 2900 50  0000 C CNN
@@
 $EndComp
 $Comp
-L PWR_FLAG #FLG052
+L PWR_FLAG #FLG050
 U 1 1 58CB39EE
 P 5100 3600
-AR Path="/592ADBF2/58CB39EE" Ref="#FLG052"  Part="1"
-AR Path="/59347BCD/58CB39EE" Ref="#FLG060"  Part="1"
-F 0 "#FLG060" H 5100 3695 50  0001 C CNN
+AR Path="/592ADBF2/58CB39EE" Ref="#FLG050"  Part="1"
+AR Path="/59347BCD/58CB39EE" Ref="#FLG058"  Part="1"
+F 0 "#FLG058" H 5100 3695 50  0001 C CNN
 F 1 "PWR_FLAG" H 5100 3780 50  0000 C CNN
 F 2 "" H 5100 3600 50  0000 C CNN
@@
 $EndComp
 $Comp
-L +3.3V #PWR053
+L +3.3V #PWR051
 U 1 1 589CCACF
 P 4100 2900
-AR Path="/592ADBF2/589CCACF" Ref="#PWR053"  Part="1"
-AR Path="/59347BCD/589CCACF" Ref="#PWR061"  Part="1"
-F 0 "#PWR061" H 4100 2750 50  0001 C CNN
+AR Path="/592ADBF2/589CCACF" Ref="#PWR051"  Part="1"
+AR Path="/59347BCD/589CCACF" Ref="#PWR059"  Part="1"
+F 0 "#PWR059" H 4100 2750 50  0001 C CNN
 F 1 "+3.3V" H 4100 3040 50  0000 C CNN
 F 2 "" H 4100 2900 50  0000 C CNN
@@
 	4100 3500 4200 3500
 $Comp
-L C_Small C16
+L C_Small C10
 U 1 1 592A96DD
 P 5700 2900
-AR Path="/592ADBF2/592A96DD" Ref="C16"  Part="1"
-AR Path="/59347BCD/592A96DD" Ref="C19"  Part="1"
-F 0 "C19" H 5710 2970 50  0000 L CNN
+AR Path="/592ADBF2/592A96DD" Ref="C10"  Part="1"
+AR Path="/59347BCD/592A96DD" Ref="C13"  Part="1"
+F 0 "C13" H 5710 2970 50  0000 L CNN
 F 1 "0.1u" H 5710 2820 50  0000 L CNN
 F 2 "Capacitors_SMD:C_0201" H 5700 2900 50  0001 C CNN
@@
 NoConn ~ 6800 3000
 $Comp
-L AS5048A U6
+L AS5048A U4
 U 1 1 5933FF2E
 P 6400 2900
-AR Path="/592ADBF2/5933FF2E" Ref="U6"  Part="1"
-AR Path="/59347BCD/5933FF2E" Ref="U8"  Part="1"
-F 0 "U8" H 6400 3450 60  0000 C CNN
+AR Path="/592ADBF2/5933FF2E" Ref="U4"  Part="1"
+AR Path="/59347BCD/5933FF2E" Ref="U6"  Part="1"
+F 0 "U6" H 6400 3450 60  0000 C CNN
 F 1 "AS5048A" H 6400 3300 60  0000 C CNN
 F 2 "mouse:TSSOP-14_4.4x5mm_Pitch0.65mm" H 6400 3300 60  0001 C CNN
@@
 F 0 "P10" H 4800 3600 50  0000 C CNN
 F 1 "ENC_Slave" V 4900 3250 50  0000 C CNN
-F 2 "mouse:STAND_AS_SLAVE" H 4800 3250 50  0001 C CNN
+F 2 "mouse:STAND_SLAVE_06" H 4800 3250 50  0001 C CNN
 F 3 "" H 4800 3250 50  0000 C CNN
 	1    4800 3250
@@
 F 0 "P9" H 4400 3600 50  0000 C CNN
 F 1 "ENC_Host" V 4500 3250 50  0000 C CNN
-F 2 "mouse:STAND_AS_HOST" H 4400 3250 50  0001 C CNN
+F 2 "mouse:STAND_HOST_06" H 4400 3250 50  0001 C CNN
 F 3 "" H 4400 3250 50  0000 C CNN
 	1    4400 3250

Commit message: 部品を配置
Parts:
- C8: renamed from C10; footprint Capacitors_SMD:C_0201 -> Capacitors_SMD:C_0201_NoSilk
Changed lines of the file:
@@
 $Descr A4 11693 8268
 encoding utf-8
-Sheet 9 15
+Sheet 10 16
 Title ""
 Date ""
@@
 $EndDescr
 $Comp
-L GND #PWR048
+L GND #PWR046
 U 1 1 589E94E9
 P 4100 3600
-AR Path="/592ADBF2/589E94E9" Ref="#PWR048"  Part="1"
-AR Path="/59347BCD/589E94E9" Ref="#PWR056"  Part="1"
-F 0 "#PWR056" H 4100 3350 50  0001 C CNN
+AR Path="/592ADBF2/589E94E9" Ref="#PWR046"  Part="1"
+AR Path="/59347BCD/589E94E9" Ref="#PWR054"  Part="1"
+F 0 "#PWR054" H 4100 3350 50  0001 C CNN
 F 1 "GND" H 4100 3450 50  0000 C CNN
 F 2 "" H 4100 3600 50  0000 C CNN
@@
 CS
 $Comp
-L PWR_FLAG #FLG049
+L PWR_FLAG #FLG047
 U 1 1 58CB39A3
 P 5100 2900
-AR Path="/592ADBF2/58CB39A3" Ref="#FLG049"  Part="1"
-AR Path="/59347BCD/58CB39A3" Ref="#FLG057"  Part="1"
-F 0 "#FLG057" H 5100 2995 50  0001 C CNN
+AR Path="/592ADBF2/58CB39A3" Ref="#FLG047"  Part="1"
+AR Path="/59347BCD/58CB39A3" Ref="#FLG055"  Part="1"
+F 0 "#FLG055" H 5100 2995 50  0001 C CNN
 F 1 "PWR_FLAG" H 5100 3080 50  0000 C CNN
 F 2 "" H 5100 2900 50  0000 C CNN
@@
 $EndComp
 $Comp
-L PWR_FLAG #FLG050
+L PWR_FLAG #FLG048
 U 1 1 58CB39EE
 P 5100 3600
-AR Path="/592ADBF2/58CB39EE" Ref="#FLG050"  Part="1"
-AR Path="/59347BCD/58CB39EE" Ref="#FLG058"  Part="1"
-F 0 "#FLG058" H 5100 3695 50  0001 C CNN
+AR Path="/592ADBF2/58CB39EE" Ref="#FLG048"  Part="1"
+AR Path="/59347BCD/58CB39EE" Ref="#FLG056"  Part="1"
+F 0 "#FLG056" H 5100 3695 50  0001 C CNN
 F 1 "PWR_FLAG" H 5100 3780 50  0000 C CNN
 F 2 "" H 5100 3600 50  0000 C CNN
@@
 $EndComp
 $Comp
-L +3.3V #PWR051
+L +3.3V #PWR049
 U 1 1 589CCACF
 P 4100 2900
-AR Path="/592ADBF2/589CCACF" Ref="#PWR051"  Part="1"
-AR Path="/59347BCD/589CCACF" Ref="#PWR059"  Part="1"
-F 0 "#PWR059" H 4100 2750 50  0001 C CNN
+AR Path="/592ADBF2/589CCACF" Ref="#PWR049"  Part="1"
+AR Path="/59347BCD/589CCACF" Ref="#PWR057"  Part="1"
+F 0 "#PWR057" H 4100 2750 50  0001 C CNN
 F 1 "+3.3V" H 4100 3040 50  0000 C CNN
 F 2 "" H 4100 2900 50  0000 C CNN
@@
 	4100 3500 4200 3500
 $Comp
-L C_Small C10
+L C_Small C8
 U 1 1 592A96DD
 P 5700 2900
-AR Path="/592ADBF2/592A96DD" Ref="C10"  Part="1"
-AR Path="/59347BCD/592A96DD" Ref="C13"  Part="1"
-F 0 "C13" H 5710 2970 50  0000 L CNN
+AR Path="/592ADBF2/592A96DD" Ref="C8"  Part="1"
+AR Path="/59347BCD/592A96DD" Ref="C11"  Part="1"
+F 0 "C11" H 5710 2970 50  0000 L CNN
 F 1 "0.1u" H 5710 2820 50  0000 L CNN
-F 2 "Capacitors_SMD:C_0201" H 5700 2900 50  0001 C CNN
+F 2 "Capacitors_SMD:C_0201_NoSilk" H 5700 2900 50  0001 C CNN
 F 3 "" H 5700 2900 50  0000 C CNN
 	1    5700 2900

Commit message: 部品を配置 kicad5
Parts:
- removed P5: ENC_Host, mouse:STAND_HOST_06, symbol CONN_01X06
- removed P6: ENC_Slave, mouse:STAND_SLAVE_06, symbol CONN_01X06
- added J10: ENC_Slave, mouse:STAND_SLAVE_06, symbol Connector:Conn_01x06_Male
- added J9: ENC_Host, mouse:STAND_HOST_06, symbol Connector:Conn_01x06_Female
- C8: symbol C_Small -> Device:C_Small
- U4: symbol AS5048A -> KERISE:AS5048A
Connections:
- wire segments 32 -> 41

Commit message: 回路にMA702を追加
Parts:
- removed U4: AS5048A, mouse:TSSOP-14_4.4x5mm_Pitch0.65mm, symbol KERISE:AS5048A
- added U4: MA702, mouse:MA702, symbol KERISE:MA702
- C8: value 0.1u -> 1u; footprint Capacitors_SMD:C_0201_NoSilk -> Capacitors_SMD:C_0402_NoSilk
Connections:
- wire segments 41 -> 22
- no-connect marks 1 -> 8
Other:
- note added: "Encoder"
Changed lines of the file:
@@
 AR Path="/592ADBF2/589E94E9" Ref="#PWR044"  Part="1"
 AR Path="/59347BCD/589E94E9" Ref="#PWR046"  Part="1"
-F 0 "#PWR046" H 4100 3350 50  0001 C CNN
+F 0 "#PWR044" H 4100 3350 50  0001 C CNN
 F 1 "GND" H 4100 3450 50  0000 C CNN
 F 2 "" H 4100 3600 50  0000 C CNN
@@
 AR Path="/592ADBF2/58CB39A3" Ref="#FLG04"  Part="1"
 AR Path="/59347BCD/58CB39A3" Ref="#FLG06"  Part="1"
-F 0 "#FLG06" H 5200 2995 50  0001 C CNN
+F 0 "#FLG04" H 5200 2995 50  0001 C CNN
 F 1 "PWR_FLAG" H 5200 3080 50  0000 C CNN
 F 2 "" H 5200 2900 50  0000 C CNN
@@
 AR Path="/592ADBF2/58CB39EE" Ref="#FLG05"  Part="1"
 AR Path="/59347BCD/58CB39EE" Ref="#FLG07"  Part="1"
-F 0 "#FLG07" H 5200 3695 50  0001 C CNN
+F 0 "#FLG05" H 5200 3695 50  0001 C CNN
 F 1 "PWR_FLAG" H 5200 3780 50  0000 C CNN
 F 2 "" H 5200 3600 50  0000 C CNN
@@
 AR Path="/592ADBF2/589CCACF" Ref="#PWR043"  Part="1"
 AR Path="/59347BCD/589CCACF" Ref="#PWR045"  Part="1"
-F 0 "#PWR045" H 4100 2750 50  0001 C CNN
+F 0 "#PWR043" H 4100 2750 50  0001 C CNN
 F 1 "+3.3V" H 4100 3040 50  0000 C CNN
 F 2 "" H 4100 2900 50  0000 C CNN
@@
 Wire Wire Line
 	4100 3500 4200 3500
-$Comp
-L Device:C_Small C8
-U 1 1 592A96DD
-P 5800 2900
-AR Path="/592ADBF2/592A96DD" Ref="C8"  Part="1"
-AR Path="/59347BCD/592A96DD" Ref="C9"  Part="1"
-F 0 "C9" H 5810 2970 50  0000 L CNN
-F 1 "0.1u" H 5810 2820 50  0000 L CNN
-F 2 "Capacitors_SMD:C_0201_NoSilk" H 5800 2900 50  0001 C CNN
-F 3 "" H 5800 2900 50  0000 C CNN
-	1    5800 2900
-	1    0    0    -1
-$EndComp
 Wire Wire Line
 	5200 3600 5200 3500
@@
 Wire Wire Line
 	5200 3200 5100 3200
-Wire Wire Line
-	5800 2500 5800 2600
-Wire Wire Line
-	5800 2700 6100 2700
-Connection ~ 5800 2700
-Wire Wire Line
-	6100 2600 5800 2600
-Connection ~ 5800 2600
-Wire Wire Line
-	5800 3000 5800 3600
-Wire Wire Line
-	5800 3600 6000 3600
-Wire Wire Line
-	6000 2900 6000 3000
-Wire Wire Line
-	6000 3300 6100 3300
-Connection ~ 6000 3400
-Wire Wire Line
-	6100 3200 6000 3200
-Connection ~ 6000 3300
-Wire Wire Line
-	6000 3100 6100 3100
-Connection ~ 6000 3200
-Wire Wire Line
-	6000 3000 6100 3000
-Connection ~ 6000 3100
-Wire Wire Line
-	6000 2900 6100 2900
-Connection ~ 6000 3000
-Wire Wire Line
-	6000 3400 6100 3400
-Connection ~ 6000 3600
-Connection ~ 5800 3600
-Wire Wire Line
-	7000 2600 6900 2600
-Wire Wire Line
-	7000 2700 6900 2700
-Wire Wire Line
-	7000 2900 6900 2900
-Wire Wire Line
-	6900 2800 7000 2800
-NoConn ~ 6900 3000
-$Comp
-L KERISE:AS5048A U4
-U 1 1 5933FF2E
-P 6500 2900
-AR Path="/592ADBF2/5933FF2E" Ref="U4"  Part="1"
-AR Path="/59347BCD/5933FF2E" Ref="U5"  Part="1"
-F 0 "U5" H 6500 3450 60  0000 C CNN
-F 1 "AS5048A" H 6500 3300 60  0000 C CNN
-F 2 "mouse:TSSOP-14_4.4x5mm_Pitch0.65mm" H 6500 3300 60  0001 C CNN
-F 3 "" H 6500 3300 60  0000 C CNN
-	1    6500 2900
-	1    0    0    -1
-$EndComp
 Text Label 5200 3500 0    60   ~ 0
 s_GND
-Text Label 5800 2500 0    60   ~ 0
-s_VDD
-Text Label 5800 3700 0    60   ~ 0
-s_GND
-Text Label 7000 2600 0    60   ~ 0
-s_CS
-Text Label 7000 2700 0    60   ~ 0
-s_SCLK
-Text Label 7000 2800 0    60   ~ 0
-s_MISO
-Text Label 7000 2900 0    60   ~ 0
-s_MOSI
 Text Label 5200 3100 0    60   ~ 0
 s_CS
@@
 Wire Wire Line
 	4200 3100 4100 3100
-Wire Wire Line
-	5800 2700 5800 2800
-Wire Wire Line
-	5800 2600 5800 2700
-Wire Wire Line
-	6000 3400 6000 3600
-Wire Wire Line
-	6000 3300 6000 3400
-Wire Wire Line
-	6000 3200 6000 3300
-Wire Wire Line
-	6000 3100 6000 3200
-Wire Wire Line
-	6000 3000 6000 3100
-Wire Wire Line
-	6000 3600 6100 3600
-Wire Wire Line
-	5800 3600 5800 3700
 $Comp
 L Connector:Conn_01x06_Female J9
@@
 AR Path="/592ADBF2/5B6F84B0" Ref="J9"  Part="1"
 AR Path="/59347BCD/5B6F84B0" Ref="J11"  Part="1"
-F 0 "J11" H 4427 3176 50  0000 L CNN
+F 0 "J9" H 4427 3176 50  0000 L CNN
 F 1 "ENC_Host" H 4427 3085 50  0000 L CNN
 F 2 "mouse:STAND_HOST_06" H 4400 3200 50  0001 C CNN
@@
 AR Path="/592ADBF2/5B6F8513" Ref="J10"  Part="1"
 AR Path="/59347BCD/5B6F8513" Ref="J12"  Part="1"
-F 0 "J12" H 5006 3578 50  0000 C CNN
+F 0 "J10" H 5006 3578 50  0000 C CNN
 F 1 "ENC_Slave" H 5006 3487 50  0000 C CNN
 F 2 "mouse:STAND_SLAVE_06" H 4900 3200 50  0001 C CNN
@@
 	1    0    0    -1
 $EndComp
+$Comp
+L KERISE:MA702 U4
+U 1 1 5B900CDD
+P 6500 2900
+AR Path="/592ADBF2/5B900CDD" Ref="U4"  Part="1"
+AR Path="/59347BCD/5B900CDD" Ref="U5"  Part="1"
+F 0 "U4" H 6500 3587 60  0000 C CNN
+F 1 "MA702" H 6500 3481 60  0000 C CNN
+F 2 "mouse:MA702" H 6500 3300 60  0001 C CNN
+F 3 "" H 6500 3300 60  0000 C CNN
+	1    6500 2900
+	1    0    0    -1
+$EndComp
+$Comp
+L Device:C_Small C8
+U 1 1 5B900E09
+P 6000 3100
+AR Path="/592ADBF2/5B900E09" Ref="C8"  Part="1"
+AR Path="/59347BCD/5B900E09" Ref="C9"  Part="1"
+F 0 "C8" H 6092 3146 50  0000 L CNN
+F 1 "1u" H 6092 3055 50  0000 L CNN
+F 2 "Capacitors_SMD:C_0402_NoSilk" H 6000 3100 50  0001 C CNN
+F 3 "~" H 6000 3100 50  0001 C CNN
+	1    6000 3100
+	1    0    0    -1
+$EndComp
+Wire Wire Line
+	6000 3000 6000 2600
+Wire Wire Line
+	6000 2600 6100 2600
+Wire Wire Line
+	6000 3200 6000 3600
+Wire Wire Line
+	6000 3600 6100 3600
+Wire Wire Line
+	6000 3600 6000 3700
+Wire Wire Line
+	6000 3700 6100 3700
+Connection ~ 6000 3600
+Text Label 6000 3700 2    60   ~ 0
+s_GND
+Text Label 6000 2600 2    60   ~ 0
+s_VDD
+Text Label 6900 3300 0    60   ~ 0
+s_CS
+Text Label 6900 3000 0    60   ~ 0
+s_SCLK
+Text Label 6900 3200 0    60   ~ 0
+s_MISO
+Text Label 6900 3100 0    60   ~ 0
+s_MOSI
+NoConn ~ 6900 2600
+NoConn ~ 6900 2700
+NoConn ~ 6900 2800
+NoConn ~ 6900 2900
+NoConn ~ 6900 3400
+NoConn ~ 6900 3500
+NoConn ~ 6900 3600
+NoConn ~ 6900 3700
+Text Notes 3900 2400 0    100  ~ 0
+Encoder
 $EndSCHEMATC

Commit message: コンデンサを追加
Parts:
- renumbered C8 to C9
Changed lines of the file:
@@
 $EndDescr
 $Comp
-L power:GND #PWR044
+L power:GND #PWR046
 U 1 1 589E94E9
 P 4100 3600
-AR Path="/592ADBF2/589E94E9" Ref="#PWR044"  Part="1"
-AR Path="/59347BCD/589E94E9" Ref="#PWR046"  Part="1"
-F 0 "#PWR044" H 4100 3350 50  0001 C CNN
+AR Path="/592ADBF2/589E94E9" Ref="#PWR046"  Part="1"
+AR Path="/59347BCD/589E94E9" Ref="#PWR048"  Part="1"
+F 0 "#PWR048" H 4100 3350 50  0001 C CNN
 F 1 "GND" H 4100 3450 50  0000 C CNN
 F 2 "" H 4100 3600 50  0000 C CNN
@@
 AR Path="/592ADBF2/58CB39A3" Ref="#FLG04"  Part="1"
 AR Path="/59347BCD/58CB39A3" Ref="#FLG06"  Part="1"
-F 0 "#FLG04" H 5200 2995 50  0001 C CNN
+F 0 "#FLG06" H 5200 2995 50  0001 C CNN
 F 1 "PWR_FLAG" H 5200 3080 50  0000 C CNN
 F 2 "" H 5200 2900 50  0000 C CNN
@@
 AR Path="/592ADBF2/58CB39EE" Ref="#FLG05"  Part="1"
 AR Path="/59347BCD/58CB39EE" Ref="#FLG07"  Part="1"
-F 0 "#FLG05" H 5200 3695 50  0001 C CNN
+F 0 "#FLG07" H 5200 3695 50  0001 C CNN
 F 1 "PWR_FLAG" H 5200 3780 50  0000 C CNN
 F 2 "" H 5200 3600 50  0000 C CNN
@@
 $EndComp
 $Comp
-L power:+3.3V #PWR043
+L power:+3.3V #PWR045
 U 1 1 589CCACF
 P 4100 2900
-AR Path="/592ADBF2/589CCACF" Ref="#PWR043"  Part="1"
-AR Path="/59347BCD/589CCACF" Ref="#PWR045"  Part="1"
-F 0 "#PWR043" H 4100 2750 50  0001 C CNN
+AR Path="/592ADBF2/589CCACF" Ref="#PWR045"  Part="1"
+AR Path="/59347BCD/589CCACF" Ref="#PWR047"  Part="1"
+F 0 "#PWR047" H 4100 2750 50  0001 C CNN
 F 1 "+3.3V" H 4100 3040 50  0000 C CNN
 F 2 "" H 4100 2900 50  0000 C CNN
@@
 AR Path="/592ADBF2/5B6F84B0" Ref="J9"  Part="1"
 AR Path="/59347BCD/5B6F84B0" Ref="J11"  Part="1"
-F 0 "J9" H 4427 3176 50  0000 L CNN
+F 0 "J11" H 4427 3176 50  0000 L CNN
 F 1 "ENC_Host" H 4427 3085 50  0000 L CNN
 F 2 "mouse:STAND_HOST_06" H 4400 3200 50  0001 C CNN
@@
 AR Path="/592ADBF2/5B6F8513" Ref="J10"  Part="1"
 AR Path="/59347BCD/5B6F8513" Ref="J12"  Part="1"
-F 0 "J10" H 5006 3578 50  0000 C CNN
+F 0 "J12" H 5006 3578 50  0000 C CNN
 F 1 "ENC_Slave" H 5006 3487 50  0000 C CNN
 F 2 "mouse:STAND_SLAVE_06" H 4900 3200 50  0001 C CNN
@@
 AR Path="/592ADBF2/5B900CDD" Ref="U4"  Part="1"
 AR Path="/59347BCD/5B900CDD" Ref="U5"  Part="1"
-F 0 "U4" H 6500 3587 60  0000 C CNN
+F 0 "U5" H 6500 3587 60  0000 C CNN
 F 1 "MA702" H 6500 3481 60  0000 C CNN
 F 2 "mouse:MA702" H 6500 3300 60  0001 C CNN
@@
 $EndComp
 $Comp
-L Device:C_Small C8
+L Device:C_Small C9
 U 1 1 5B900E09
 P 6000 3100
-AR Path="/592ADBF2/5B900E09" Ref="C8"  Part="1"
-AR Path="/59347BCD/5B900E09" Ref="C9"  Part="1"
-F 0 "C8" H 6092 3146 50  0000 L CNN
+AR Path="/592ADBF2/5B900E09" Ref="C9"  Part="1"
+AR Path="/59347BCD/5B900E09" Ref="C10"  Part="1"
+F 0 "C10" H 6092 3146 50  0000 L CNN
 F 1 "1u" H 6092 3055 50  0000 L CNN
 F 2 "Capacitors_SMD:C_0402_NoSilk" H 6000 3100 50  0001 C CNN

Commit message: KERISEv4-5に向けて回路図を更新
Parts:
- removed C9: 1u, Capacitors_SMD:C_0402_NoSilk, symbol Device:C_Small
- removed U4: MA702, mouse:MA702, symbol KERISE:MA702
- added C10: 0.1u, symbol Device:C_Small
- added U4: AS5048A, symbol KERISE:AS5048A
Connections:
- wire segments 22 -> 35
- no-connect marks 8 -> 1
Changed lines of the file:
@@
 $Descr A4 11693 8268
 encoding utf-8
-Sheet 9 14
+Sheet 9 15
 Title ""
 Date ""
@@
 $EndDescr
 $Comp
-L power:GND #PWR046
+L power:GND #PWR048
 U 1 1 589E94E9
 P 4100 3600
-AR Path="/592ADBF2/589E94E9" Ref="#PWR046"  Part="1"
-AR Path="/59347BCD/589E94E9" Ref="#PWR048"  Part="1"
-F 0 "#PWR048" H 4100 3350 50  0001 C CNN
+AR Path="/592ADBF2/589E94E9" Ref="#PWR048"  Part="1"
+AR Path="/59347BCD/589E94E9" Ref="#PWR050"  Part="1"
+F 0 "#PWR050" H 4100 3350 50  0001 C CNN
 F 1 "GND" H 4100 3450 50  0000 C CNN
 F 2 "" H 4100 3600 50  0000 C CNN
@@
 $EndComp
 $Comp
-L power:+3.3V #PWR045
+L power:+3.3V #PWR047
 U 1 1 589CCACF
 P 4100 2900
-AR Path="/592ADBF2/589CCACF" Ref="#PWR045"  Part="1"
-AR Path="/59347BCD/589CCACF" Ref="#PWR047"  Part="1"
-F 0 "#PWR047" H 4100 2750 50  0001 C CNN
+AR Path="/592ADBF2/589CCACF" Ref="#PWR047"  Part="1"
+AR Path="/59347BCD/589CCACF" Ref="#PWR049"  Part="1"
+F 0 "#PWR049" H 4100 2750 50  0001 C CNN
 F 1 "+3.3V" H 4100 3040 50  0000 C CNN
 F 2 "" H 4100 2900 50  0000 C CNN
@@
 	1    0    0    -1
 $EndComp
-$Comp
-L KERISE:MA702 U4
-U 1 1 5B900CDD
-P 6500 2900
-AR Path="/592ADBF2/5B900CDD" Ref="U4"  Part="1"
-AR Path="/59347BCD/5B900CDD" Ref="U5"  Part="1"
-F 0 "U5" H 6500 3587 60  0000 C CNN
-F 1 "MA702" H 6500 3481 60  0000 C CNN
-F 2 "mouse:MA702" H 6500 3300 60  0001 C CNN
-F 3 "" H 6500 3300 60  0000 C CNN
-	1    6500 2900
-	1    0    0    -1
-$EndComp
-$Comp
-L Device:C_Small C9
-U 1 1 5B900E09
-P 6000 3100
-AR Path="/592ADBF2/5B900E09" Ref="C9"  Part="1"
-AR Path="/59347BCD/5B900E09" Ref="C10"  Part="1"
-F 0 "C10" H 6092 3146 50  0000 L CNN
-F 1 "1u" H 6092 3055 50  0000 L CNN
-F 2 "Capacitors_SMD:C_0402_NoSilk" H 6000 3100 50  0001 C CNN
-F 3 "~" H 6000 3100 50  0001 C CNN
-	1    6000 3100
-	1    0    0    -1
-$EndComp
-Wire Wire Line
-	6000 3000 6000 2600
-Wire Wire Line
-	6000 2600 6100 2600
-Wire Wire Line
-	6000 3200 6000 3600
-Wire Wire Line
-	6000 3600 6100 3600
-Wire Wire Line
-	6000 3600 6000 3700
-Wire Wire Line
-	6000 3700 6100 3700
-Connection ~ 6000 3600
-Text Label 6000 3700 2    60   ~ 0
-s_GND
-Text Label 6000 2600 2    60   ~ 0
-s_VDD
-Text Label 6900 3300 0    60   ~ 0
-s_CS
-Text Label 6900 3000 0    60   ~ 0
-s_SCLK
-Text Label 6900 3200 0    60   ~ 0
-s_MISO
-Text Label 6900 3100 0    60   ~ 0
-s_MOSI
-NoConn ~ 6900 2600
-NoConn ~ 6900 2700
-NoConn ~ 6900 2800
-NoConn ~ 6900 2900
-NoConn ~ 6900 3400
-NoConn ~ 6900 3500
-NoConn ~ 6900 3600
-NoConn ~ 6900 3700
 Text Notes 3900 2400 0    100  ~ 0
 Encoder
+$Comp
+L KERISE:AS5048A U4
+U 1 1 5C2A3915
+P 6900 3000
+AR Path="/592ADBF2/5C2A3915" Ref="U4"  Part="1"
+AR Path="/59347BCD/5C2A3915" Ref="U5"  Part="1"
+F 0 "U5" H 6900 3687 60  0000 C CNN
+F 1 "AS5048A" H 6900 3581 60  0000 C CNN
+F 2 "" H 6900 3400 60  0000 C CNN
+F 3 "" H 6900 3400 60  0000 C CNN
+	1    6900 3000
+	1    0    0    -1
+$EndComp
+Text Label 6100 2700 2    60   ~ 0
+s_VDD
+$Comp
+L Device:C_Small C10
+U 1 1 5C2A3C19
+P 6100 3000
+AR Path="/592ADBF2/5C2A3C19" Ref="C10"  Part="1"
+AR Path="/59347BCD/5C2A3C19" Ref="C11"  Part="1"
+F 0 "C11" H 6192 3046 50  0000 L CNN
+F 1 "0.1u" H 6192 2955 50  0000 L CNN
+F 2 "" H 6100 3000 50  0001 C CNN
+F 3 "~" H 6100 3000 50  0001 C CNN
+	1    6100 3000
+	1    0    0    -1
+$EndComp
+Wire Wire Line
+	6500 3000 6400 3000
+Wire Wire Line
+	6400 3000 6400 3100
+Wire Wire Line
+	6400 3100 6500 3100
+Wire Wire Line
+	6400 3100 6400 3200
+Wire Wire Line
+	6400 3200 6500 3200
+Connection ~ 6400 3100
+Wire Wire Line
+	6500 3300 6400 3300
+Wire Wire Line
+	6400 3300 6400 3200
+Connection ~ 6400 3200
+Wire Wire Line
+	6500 3400 6400 3400
+Wire Wire Line
+	6400 3400 6400 3300
+Connection ~ 6400 3300
+Wire Wire Line
+	6500 3500 6400 3500
+Wire Wire Line
+	6400 3500 6400 3400
+Connection ~ 6400 3400
+Wire Wire Line
+	6500 3700 6400 3700
+Wire Wire Line
+	6400 3700 6400 3500
+Connection ~ 6400 3500
+Wire Wire Line
+	6400 3700 6100 3700
+Wire Wire Line
+	6100 3700 6100 3100
+Connection ~ 6400 3700
+Wire Wire Line
+	6500 2800 6100 2800
+Wire Wire Line
+	6100 2800 6100 2900
+Wire Wire Line
+	6500 2700 6100 2700
+Wire Wire Line
+	6100 2700 6100 2800
+Connection ~ 6100 2800
+Text Label 6100 3700 2    60   ~ 0
+s_GND
+NoConn ~ 7300 3100
+Text Label 7300 2700 0    60   ~ 0
+s_CS
+Text Label 7300 2900 0    60   ~ 0
+s_MISO
+Text Label 7300 3000 0    60   ~ 0
+s_MOSI
+Text Label 7300 2800 0    60   ~ 0
+s_SCLK
 $EndSCHEMATC
