File: kicad/Fan.sch (KiCad schematic (older format))
At the start: 3 parts, among them P4 Fan, Q3 DMN3065LW-7

Commit message: 回路を改良
受光部をフォトトランジスタに変更
測距センサをVL6180Xに変更
動作電圧を3Vに変更
Parts:
- renumbered Q3 to Q5, R15 to R10
Changed lines of the file:
@@
 LIBS:ftdi
 LIBS:gennum
-LIBS:graphic
 LIBS:hc11
 LIBS:ir
 LIBS:Lattice
 LIBS:leds
-LIBS:logo
 LIBS:maxim
 LIBS:mechanical
@@
 LIBS:zetex
 LIBS:Zilog
+LIBS:graphic_symbols
+LIBS:infineon
+LIBS:intersil
+LIBS:LEM
+LIBS:logic_programmable
+LIBS:RFSolutions
 LIBS:KERISE-cache
 EELAYER 25 0
@@
 $EndDescr
 $Comp
-L Q_NMOS_GSD Q3
+L Q_NMOS_GSD Q5
 U 1 1 58AB90D4
 P 5050 4800
-F 0 "Q3" H 5350 4850 50  0000 R CNN
+F 0 "Q5" H 5350 4850 50  0000 R CNN
 F 1 "DMN3065LW-7" H 5800 4750 50  0000 R CNN
 F 2 "TO_SOT_Packages_SMD:SOT-323_SC-70" H 5250 4900 50  0001 C CNN
@@
 $EndComp
 $Comp
-L GND #PWR047
+L GND #PWR045
 U 1 1 58AB90DB
 P 5150 5300
-F 0 "#PWR047" H 5150 5050 50  0001 C CNN
+F 0 "#PWR045" H 5150 5050 50  0001 C CNN
 F 1 "GND" H 5150 5150 50  0000 C CNN
 F 2 "" H 5150 5300 50  0000 C CNN
@@
 	5150 5000 5150 5300
 $Comp
-L R R15
+L R R10
 U 1 1 58AB90F7
 P 4750 5050
-F 0 "R15" V 4830 5050 50  0000 C CNN
+F 0 "R10" V 4830 5050 50  0000 C CNN
 F 1 "10k" V 4750 5050 50  0000 C CNN
 F 2 "Resistors_SMD:R_0201" V 4680 5050 50  0001 C CNN
@@
 Connection ~ 4750 4800
 $Comp
-L GND #PWR048
+L GND #PWR046
 U 1 1 58AB9100
 P 4750 5300
-F 0 "#PWR048" H 4750 5050 50  0001 C CNN
+F 0 "#PWR046" H 4750 5050 50  0001 C CNN
 F 1 "GND" H 4750 5150 50  0000 C CNN
 F 2 "" H 4750 5300 50  0000 C CNN
@@
 $EndComp
 $Comp
-L +BATT #PWR049
+L +BATT #PWR047
 U 1 1 58AB927D
 P 5150 4100
-F 0 "#PWR049" H 5150 3950 50  0001 C CNN
+F 0 "#PWR047" H 5150 3950 50  0001 C CNN
 F 1 "+BATT" H 5150 4240 50  0000 C CNN
 F 2 "" H 5150 4100 50  0000 C CNN

Commit message: 部品を配置
Parts:
- R10: footprint Resistors_SMD:R_0201 -> Resistors_SMD:R_0201_NoSilk
- renumbered Q5 to Q7
Changed lines of the file:
@@
 $Descr A4 11693 8268
 encoding utf-8
-Sheet 8 15
+Sheet 7 16
 Title ""
 Date ""
@@
 $EndDescr
 $Comp
-L Q_NMOS_GSD Q5
+L Q_NMOS_GSD Q7
 U 1 1 58AB90D4
 P 5050 4800
-F 0 "Q5" H 5350 4850 50  0000 R CNN
+F 0 "Q7" H 5350 4850 50  0000 R CNN
 F 1 "DMN3065LW-7" H 5800 4750 50  0000 R CNN
 F 2 "TO_SOT_Packages_SMD:SOT-323_SC-70" H 5250 4900 50  0001 C CNN
@@
 $EndComp
 $Comp
-L GND #PWR045
+L GND #PWR043
 U 1 1 58AB90DB
 P 5150 5300
-F 0 "#PWR045" H 5150 5050 50  0001 C CNN
+F 0 "#PWR043" H 5150 5050 50  0001 C CNN
 F 1 "GND" H 5150 5150 50  0000 C CNN
 F 2 "" H 5150 5300 50  0000 C CNN
@@
 F 0 "R10" V 4830 5050 50  0000 C CNN
 F 1 "10k" V 4750 5050 50  0000 C CNN
-F 2 "Resistors_SMD:R_0201" V 4680 5050 50  0001 C CNN
+F 2 "Resistors_SMD:R_0201_NoSilk" V 4680 5050 50  0001 C CNN
 F 3 "" H 4750 5050 50  0000 C CNN
 	1    4750 5050
@@
 Connection ~ 4750 4800
 $Comp
-L GND #PWR046
+L GND #PWR044
 U 1 1 58AB9100
 P 4750 5300
-F 0 "#PWR046" H 4750 5050 50  0001 C CNN
+F 0 "#PWR044" H 4750 5050 50  0001 C CNN
 F 1 "GND" H 4750 5150 50  0000 C CNN
 F 2 "" H 4750 5300 50  0000 C CNN
@@
 $EndComp
 $Comp
-L +BATT #PWR047
+L +BATT #PWR045
 U 1 1 58AB927D
 P 5150 4100
-F 0 "#PWR047" H 5150 3950 50  0001 C CNN
+F 0 "#PWR045" H 5150 3950 50  0001 C CNN
 F 1 "+BATT" H 5150 4240 50  0000 C CNN
 F 2 "" H 5150 4100 50  0000 C CNN

Commit message: 部品を配置 kicad5
Parts:
- removed P4: Fan, mouse:SMD_conn_2, symbol CONN_01X02
- added J8: Fan, mouse:SMD_conn_2, symbol Connector_Generic:Conn_01x02
- Q7: symbol Q_NMOS_GSD -> Device:Q_NMOS_GSD
- R10: symbol R -> Device:R
Connections:
- net +BATT: now also J8.1 (Pin_1)
- net fan_to_fet: now also J8.2 (Pin_2)
Changed lines of the file:
@@
-EESchema Schematic File Version 2
-LIBS:power
-LIBS:device
-LIBS:transistors
-LIBS:conn
-LIBS:linear
-LIBS:regul
-LIBS:74xx
-LIBS:cmos4000
-LIBS:adc-dac
-LIBS:memory
-LIBS:xilinx
-LIBS:microcontrollers
-LIBS:dsp
-LIBS:microchip
-LIBS:analog_switches
-LIBS:motorola
-LIBS:texas
-LIBS:intel
-LIBS:audio
-LIBS:interface
-LIBS:digital-audio
-LIBS:philips
-LIBS:display
-LIBS:cypress
-LIBS:siliconi
-LIBS:opto
-LIBS:atmel
-LIBS:contrib
-LIBS:valves
-LIBS:KERISE
-LIBS:74xgxx
-LIBS:ac-dc
-LIBS:actel
-LIBS:allegro
-LIBS:Altera
-LIBS:analog_devices
-LIBS:battery_management
-LIBS:bbd
-LIBS:bosch
-LIBS:brooktre
-LIBS:cmos_ieee
-LIBS:dc-dc
-LIBS:diode
-LIBS:elec-unifil
-LIBS:ESD_Protection
-LIBS:ftdi
-LIBS:gennum
-LIBS:hc11
-LIBS:ir
-LIBS:Lattice
-LIBS:leds
-LIBS:maxim
-LIBS:mechanical
-LIBS:microchip_dspic33dsc
-LIBS:microchip_pic10mcu
-LIBS:microchip_pic12mcu
-LIBS:microchip_pic16mcu
-LIBS:microchip_pic18mcu
-LIBS:microchip_pic24mcu
-LIBS:microchip_pic32mcu
-LIBS:modules
-LIBS:motor_drivers
-LIBS:motors
-LIBS:msp430
-LIBS:nordicsemi
-LIBS:nxp
-LIBS:nxp_armmcu
-LIBS:onsemi
-LIBS:Oscillators
-LIBS:Power_Management
-LIBS:powerint
-LIBS:pspice
-LIBS:references
-LIBS:relays
-LIBS:rfcom
-LIBS:sensors
-LIBS:silabs
-LIBS:stm8
-LIBS:stm32
-LIBS:supertex
-LIBS:switches
-LIBS:transf
-LIBS:triac_thyristor
-LIBS:ttl_ieee
-LIBS:video
-LIBS:wiznet
-LIBS:Worldsemi
-LIBS:Xicor
-LIBS:zetex
-LIBS:Zilog
-LIBS:graphic_symbols
-LIBS:infineon
-LIBS:intersil
-LIBS:LEM
-LIBS:logic_programmable
-LIBS:RFSolutions
+EESchema Schematic File Version 4
 LIBS:KERISE-cache
-EELAYER 25 0
+EELAYER 26 0
 EELAYER END
 $Descr A4 11693 8268
 encoding utf-8
-Sheet 7 15
+Sheet 7 14
 Title ""
 Date ""
@@
 $EndDescr
 $Comp
-L Q_NMOS_GSD Q7
+L Device:Q_NMOS_GSD Q7
 U 1 1 58AB90D4
 P 5050 4800
@@
 	1    0    0    -1
 $EndComp
-$Comp
-L GND #PWR043
-U 1 1 58AB90DB
-P 5150 5300
-F 0 "#PWR043" H 5150 5050 50  0001 C CNN
-F 1 "GND" H 5150 5150 50  0000 C CNN
-F 2 "" H 5150 5300 50  0000 C CNN
-F 3 "" H 5150 5300 50  0000 C CNN
-	1    5150 5300
-	1    0    0    -1
-$EndComp
 Text HLabel 4550 4800 0    60   Input ~ 0
 Fan
 Wire Wire Line
-	4550 4800 4850 4800
+	4550 4800 4750 4800
 Wire Wire Line
 	5150 5000 5150 5300
 $Comp
-L R R10
+L Device:R R10
 U 1 1 58AB90F7
 P 4750 5050
@@
 Connection ~ 4750 4800
 $Comp
-L GND #PWR044
+L power:GND #PWR040
 U 1 1 58AB9100
 P 4750 5300
-F 0 "#PWR044" H 4750 5050 50  0001 C CNN
+F 0 "#PWR040" H 4750 5050 50  0001 C CNN
 F 1 "GND" H 4750 5150 50  0000 C CNN
 F 2 "" H 4750 5300 50  0000 C CNN
@@
 	4750 5300 4750 5200
 $Comp
-L CONN_01X02 P4
-U 1 1 58AB920C
-P 5450 4350
-F 0 "P4" H 5450 4500 50  0000 C CNN
-F 1 "Fan" V 5550 4350 50  0000 C CNN
-F 2 "mouse:SMD_conn_2" H 5450 4350 50  0001 C CNN
-F 3 "" H 5450 4350 50  0000 C CNN
-	1    5450 4350
-	1    0    0    -1
-$EndComp
-$Comp
-L +BATT #PWR045
+L power:+BATT #PWR041
 U 1 1 58AB927D
 P 5150 4100
-F 0 "#PWR045" H 5150 3950 50  0001 C CNN
+F 0 "#PWR041" H 5150 3950 50  0001 C CNN
 F 1 "+BATT" H 5150 4240 50  0000 C CNN
 F 2 "" H 5150 4100 50  0000 C CNN
@@
 Text Label 5150 4550 0    60   ~ 0
 fan_to_fet
+Wire Wire Line
+	4750 4800 4850 4800
+$Comp
+L Connector_Generic:Conn_01x02 J8
+U 1 1 5B6F4A9E
+P 5450 4300
+F 0 "J8" H 5530 4292 50  0000 L CNN
+F 1 "Fan" H 5530 4201 50  0000 L CNN
+F 2 "mouse:SMD_conn_2" H 5450 4300 50  0001 C CNN
+F 3 "~" H 5450 4300 50  0001 C CNN
+	1    5450 4300
+	1    0    0    -1
+$EndComp
+$Comp
+L power:GND #PWR042
+U 1 1 5B709ACC
+P 5150 5300
+F 0 "#PWR042" H 5150 5050 50  0001 C CNN
+F 1 "GND" H 5150 5150 50  0000 C CNN
+F 2 "" H 5150 5300 50  0000 C CNN
+F 3 "" H 5150 5300 50  0000 C CNN
+	1    5150 5300
+	1    0    0    -1
+$EndComp
 $EndSCHEMATC

Commit message: フットプリントを割り当て
Parts:
- R10: footprint Resistors_SMD:R_0201_NoSilk -> Resistor_SMD:R_0201_0603Metric
Changed lines of the file:
@@
 F 0 "R10" V 4830 5050 50  0000 C CNN
 F 1 "10k" V 4750 5050 50  0000 C CNN
-F 2 "Resistors_SMD:R_0201_NoSilk" V 4680 5050 50  0001 C CNN
+F 2 "Resistor_SMD:R_0201_0603Metric" V 4680 5050 50  0001 C CNN
 F 3 "" H 4750 5050 50  0000 C CNN
 	1    4750 5050
@@
 Connection ~ 4750 4800
 $Comp
-L power:GND #PWR044
+L power:GND #PWR046
 U 1 1 58AB9100
 P 4750 5300
-F 0 "#PWR044" H 4750 5050 50  0001 C CNN
+F 0 "#PWR046" H 4750 5050 50  0001 C CNN
 F 1 "GND" H 4750 5150 50  0000 C CNN
 F 2 "" H 4750 5300 50  0000 C CNN
@@
 	4750 5300 4750 5200
 $Comp
-L power:+BATT #PWR045
+L power:+BATT #PWR047
 U 1 1 58AB927D
 P 5150 4100
-F 0 "#PWR045" H 5150 3950 50  0001 C CNN
+F 0 "#PWR047" H 5150 3950 50  0001 C CNN
 F 1 "+BATT" H 5150 4240 50  0000 C CNN
 F 2 "" H 5150 4100 50  0000 C CNN
@@
 $EndComp
 $Comp
-L power:GND #PWR046
+L power:GND #PWR048
 U 1 1 5B709ACC
 P 5150 5300
-F 0 "#PWR046" H 5150 5050 50  0001 C CNN
+F 0 "#PWR048" H 5150 5050 50  0001 C CNN
 F 1 "GND" H 5150 5150 50  0000 C CNN
 F 2 "" H 5150 5300 50  0000 C CNN

Commit message: 部品を配置
Parts:
- added C13: 10u, Capacitor_SMD:C_0402_1005Metric, symbol Device:C
Connections:
- net +BATT: now also C13.1
- net GND: now also C13.2
Changed lines of the file:
@@
 	1    0    0    -1
 $EndComp
+$Comp
+L Device:C C13
+U 1 1 5C29CF10
+P 6050 4850
+F 0 "C13" H 6165 4896 50  0000 L CNN
+F 1 "10u" H 6165 4805 50  0000 L CNN
+F 2 "Capacitor_SMD:C_0402_1005Metric" H 6088 4700 50  0001 C CNN
+F 3 "~" H 6050 4850 50  0001 C CNN
+	1    6050 4850
+	1    0    0    -1
+$EndComp
+$Comp
+L power:GND #PWR050
+U 1 1 5C29CF9E
+P 6050 5300
+F 0 "#PWR050" H 6050 5050 50  0001 C CNN
+F 1 "GND" H 6050 5150 50  0000 C CNN
+F 2 "" H 6050 5300 50  0000 C CNN
+F 3 "" H 6050 5300 50  0000 C CNN
+	1    6050 5300
+	1    0    0    -1
+$EndComp
+Wire Wire Line
+	6050 5000 6050 5300
+$Comp
+L power:+BATT #PWR049
+U 1 1 5C29D01F
+P 6050 4100
+F 0 "#PWR049" H 6050 3950 50  0001 C CNN
+F 1 "+BATT" H 6050 4240 50  0000 C CNN
+F 2 "" H 6050 4100 50  0000 C CNN
+F 3 "" H 6050 4100 50  0000 C CNN
+	1    6050 4100
+	1    0    0    -1
+$EndComp
+Wire Wire Line
+	6050 4100 6050 4700
 $EndSCHEMATC
