File: kicad/Fan.sch (KiCad schematic (older format))
At the start: 4 parts, among them J8 Fan, Q7 DMN3065LW-7

Commit message: フットプリントを改良
Parts:
- Q7: footprint TO_SOT_Packages_SMD:SOT-323_SC-70 -> Package_TO_SOT_SMD:SOT-323_SC-70
Changed lines of the file:
@@
 F 0 "Q7" H 5350 4850 50  0000 R CNN
 F 1 "DMN3065LW-7" H 5800 4750 50  0000 R CNN
-F 2 "TO_SOT_Packages_SMD:SOT-323_SC-70" H 5250 4900 50  0001 C CNN
+F 2 "Package_TO_SOT_SMD:SOT-323_SC-70" H 5250 4900 50  0001 C CNN
 F 3 "" H 5050 4800 50  0000 C CNN
 	1    5050 4800
