File: kicad/KERISE.kicad_pcb (KiCad board)
At the start: 2 copper layers, 40 x 44 mm, 106 parts, among them J1 Motor_L, J10 ENC_Slave, J11 ENC_Host, J12 ENC_Slave, J13 Host, J14 Slave, J15 Host, J16 Slave, J2 Motor_R, J3 Host, J4 Slave, J5 Host, J6 Slave, J7 COM, J8 Fan, J9 ENC_Host, P1 ToF_Host, P2 ToF_Slave, Q1 MTM231232LBF, Q10 SFH3015FA, Q11 MTM231232LBF, Q12 DMN3065LW-7, Q13 SFH3015FA, Q14 DMN3065LW-7, Q2 DMN3065LW-7, Q3 SFH3015FA, Q4 MTM231232LBF, Q5 DMN3065LW-7, Q6 SFH3015FA, Q7 DMN3065LW-7, Q8 MTM231232LBF, Q9 DMN3065LW-7, SW1 RESET, SW2 UPLOAD, U1 ESP32-PICO-D4, U2 DRV8835, U3 LXDC2UR30, U4 AS5048A, U5 AS5048A, U6 ICM-20602, U7 ICM-20602, U8 PCA9632, U9 VL6180X

Commit message: 配置を改良
Parts:
- L3: footprint Capacitors_SMD:C_0603 -> Inductor_SMD:L_0603_1608Metric
- moved C1 2.12 mm to (141.5, 117.0), turned to 90 degrees
- moved D2 1.12 mm to (157.5, 90.0)
- moved D1 1.12 mm to (139.5, 90.0)
- moved R4 1.00 mm to (138.5, 90.5)
- moved R5 1.00 mm to (158.5, 90.5)
- moved C3 0.50 mm to (156.0, 118.8)
- moved R1 0.50 mm to (135.5, 97.5)
- moved R11 0.25 mm to (161.8, 115.5)
- moved R13 0.25 mm to (161.8, 106.0)
- moved R6 0.25 mm to (132.8, 106.0)
- moved R8 0.25 mm to (132.8, 115.5)
- moved U2 0.25 mm to (154.8, 116.8)
- moved D3 0.22 mm to (132.9, 105.7)
- moved D4 0.22 mm to (132.9, 115.2)
- moved D5 0.22 mm to (164.1, 115.2)
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Routing:
- net +BATT: track 36.7 -> 42.5 mm
