File: kicad/Power.sch (KiCad schematic (older format))
At the start: 13 parts, among them U3 LXDC2UR30

Commit message: リファレンスを除去
Parts:
- L3: footprint Capacitors_SMD:C_0603 -> Inductor_SMD:L_0603_1608Metric
Changed lines of the file:
@@
 F 0 "L3" H 7630 4340 50  0000 L CNN
 F 1 "100u" H 7630 4260 50  0000 L CNN
-F 2 "Capacitors_SMD:C_0603" H 7600 4300 50  0001 C CNN
+F 2 "Inductor_SMD:L_0603_1608Metric" H 7600 4300 50  0001 C CNN
 F 3 "" H 7600 4300 50  0001 C CNN
 	1    7600 4300
