File: kicad/ToF.sch (KiCad schematic (older format))
At the start: 7 parts, among them P1 ToF_Host, P2 ToF_Slave, U9 VL6180X

Commit message: フットプリントを割り当て
Parts:
- C21: renamed from C20; footprint Capacitors_SMD:C_0402_NoSilk -> Capacitor_SMD:C_0402_1005Metric
- C22: renamed from C21; footprint Capacitors_SMD:C_0201_NoSilk -> Capacitor_SMD:C_0201_0603Metric
- R20, R21: footprint Resistors_SMD:R_0201_NoSilk -> Resistor_SMD:R_0201_0603Metric
- U9: footprint (none) -> mouse:VL6180X
Changed lines of the file:
@@
 SCL
 $Comp
-L Device:C_Small C21
+L Device:C_Small C22
 U 1 1 592BA26F
 P 3900 3800
-F 0 "C21" H 3910 3870 50  0000 L CNN
+F 0 "C22" H 3910 3870 50  0000 L CNN
 F 1 "0.1u" H 3910 3720 50  0000 L CNN
-F 2 "Capacitors_SMD:C_0201_NoSilk" H 3900 3800 50  0001 C CNN
+F 2 "Capacitor_SMD:C_0201_0603Metric" H 3900 3800 50  0001 C CNN
 F 3 "" H 3900 3800 50  0000 C CNN
 	1    3900 3800
@@
 $EndComp
 $Comp
-L Device:C_Small C20
+L Device:C_Small C21
 U 1 1 592BA2BF
 P 3600 3800
-F 0 "C20" H 3610 3870 50  0000 L CNN
+F 0 "C21" H 3610 3870 50  0000 L CNN
 F 1 "4.7u" H 3610 3720 50  0000 L CNN
-F 2 "Capacitors_SMD:C_0402_NoSilk" H 3600 3800 50  0001 C CNN
+F 2 "Capacitor_SMD:C_0402_1005Metric" H 3600 3800 50  0001 C CNN
 F 3 "" H 3600 3800 50  0000 C CNN
 	1    3600 3800
@@
 F 0 "R20" V 5780 3450 50  0000 C CNN
 F 1 "4.7k" V 5700 3450 50  0000 C CNN
-F 2 "Resistors_SMD:R_0201_NoSilk" V 5630 3450 50  0001 C CNN
+F 2 "Resistor_SMD:R_0201_0603Metric" V 5630 3450 50  0001 C CNN
 F 3 "" H 5700 3450 50  0001 C CNN
 	1    5700 3450
@@
 F 0 "R21" V 5980 3450 50  0000 C CNN
 F 1 "4.7k" V 5900 3450 50  0000 C CNN
-F 2 "Resistors_SMD:R_0201_NoSilk" V 5830 3450 50  0001 C CNN
+F 2 "Resistor_SMD:R_0201_0603Metric" V 5830 3450 50  0001 C CNN
 F 3 "" H 5900 3450 50  0001 C CNN
 	1    5900 3450
@@
 	4200 3400 4200 3500
 $Comp
-L power:GND #PWR080
+L power:GND #PWR082
 U 1 1 5C29A844
 P 4300 2700
-F 0 "#PWR080" H 4300 2450 50  0001 C CNN
+F 0 "#PWR082" H 4300 2450 50  0001 C CNN
 F 1 "GND" H 4305 2527 50  0000 C CNN
 F 2 "" H 4300 2700 50  0001 C CNN
@@
 $EndComp
 $Comp
-L power:+3.3V #PWR079
+L power:+3.3V #PWR081
 U 1 1 5C29A8B4
 P 4300 2200
-F 0 "#PWR079" H 4300 2050 50  0001 C CNN
+F 0 "#PWR081" H 4300 2050 50  0001 C CNN
 F 1 "+3.3V" H 4315 2373 50  0000 C CNN
 F 2 "" H 4300 2200 50  0001 C CNN
@@
 F 0 "U9" H 4800 3587 60  0000 C CNN
 F 1 "VL6180X" H 4800 3481 60  0000 C CNN
-F 2 "" H 4800 3300 60  0000 C CNN
+F 2 "mouse:VL6180X" H 4800 3300 60  0001 C CNN
 F 3 "" H 4800 3300 60  0000 C CNN
 	1    4800 3300

Commit message: 部品を配置
Parts:
- renumbered C21 to C26, C22 to C27
Changed lines of the file:
@@
 SCL
 $Comp
-L Device:C_Small C22
+L Device:C_Small C27
 U 1 1 592BA26F
 P 3900 3800
-F 0 "C22" H 3910 3870 50  0000 L CNN
+F 0 "C27" H 3910 3870 50  0000 L CNN
 F 1 "0.1u" H 3910 3720 50  0000 L CNN
 F 2 "Capacitor_SMD:C_0201_0603Metric" H 3900 3800 50  0001 C CNN
@@
 $EndComp
 $Comp
-L Device:C_Small C21
+L Device:C_Small C26
 U 1 1 592BA2BF
 P 3600 3800
-F 0 "C21" H 3610 3870 50  0000 L CNN
+F 0 "C26" H 3610 3870 50  0000 L CNN
 F 1 "4.7u" H 3610 3720 50  0000 L CNN
 F 2 "Capacitor_SMD:C_0402_1005Metric" H 3600 3800 50  0001 C CNN
@@
 	4200 3400 4200 3500
 $Comp
-L power:GND #PWR082
+L power:GND #PWR084
 U 1 1 5C29A844
 P 4300 2700
-F 0 "#PWR082" H 4300 2450 50  0001 C CNN
+F 0 "#PWR084" H 4300 2450 50  0001 C CNN
 F 1 "GND" H 4305 2527 50  0000 C CNN
 F 2 "" H 4300 2700 50  0001 C CNN
@@
 $EndComp
 $Comp
-L power:+3.3V #PWR081
+L power:+3.3V #PWR083
 U 1 1 5C29A8B4
 P 4300 2200
-F 0 "#PWR081" H 4300 2050 50  0001 C CNN
+F 0 "#PWR083" H 4300 2050 50  0001 C CNN
 F 1 "+3.3V" H 4315 2373 50  0000 C CNN
 F 2 "" H 4300 2200 50  0001 C CNN

Commit message: LEDの抵抗を集合抵抗に変更
Parts:
- renumbered R20 to R16, R21 to R17
Changed lines of the file:
@@
 	5400 3400 5300 3400
 $Comp
-L Device:R R20
+L Device:R R16
 U 1 1 5AB6394F
 P 5700 3450
-F 0 "R20" V 5780 3450 50  0000 C CNN
+F 0 "R16" V 5780 3450 50  0000 C CNN
 F 1 "4.7k" V 5700 3450 50  0000 C CNN
 F 2 "Resistor_SMD:R_0201_0603Metric" V 5630 3450 50  0001 C CNN
@@
 $EndComp
 $Comp
-L Device:R R21
+L Device:R R17
 U 1 1 5AB639A9
 P 5900 3450
-F 0 "R21" V 5980 3450 50  0000 C CNN
+F 0 "R17" V 5980 3450 50  0000 C CNN
 F 1 "4.7k" V 5900 3450 50  0000 C CNN
 F 2 "Resistor_SMD:R_0201_0603Metric" V 5830 3450 50  0001 C CNN
